Commit message: new file:   LICENSE 	modified:   PORTING_NOTES.md 	modified:   README.md 	new file:   plan.md 	new file:   src/armv7_bringup/CMakeLists.txt 	modified:   src/armv7_bringup/config/EUPH11_config.yaml 	modified:   src/armv7_bringup/config/EUPH14_config.yaml 	modified:   src/armv7_bringup/config/EUPH17_config.yaml 	modified:   src/armv7_bringup/config/ros2_controllers.yaml 	modified:   src/armv7_bringup/launch/arm.launch.py 	new file:   src/armv7_bringup/package.xml 	modified:   src/armv7_bringup/urdf/armv7_ethercat.ros2_control.xacro 	modified:   src/armv7_description/CMakeLists.txt 	modified:   src/armv7_description/launch/display.launch.py 	modified:   src/armv7_description/launch/gazebo.launch.py 	modified:   src/armv7_description/package.xml 	modified:   src/armv7_description/urdf/armv7.csv 	modified:   src/armv7_description/urdf/armv7.urdf 	new file:   src/armv7_description/urdf/armv7.urdf.xacro 	modified:   src/armv7_moveit_config/.setup_assistant 	new file:   src/armv7_moveit_config/CMakeLists.txt 	new file:   src/armv7_moveit_config/launch/_moveit_config_loader.py 	modified:   src/armv7_moveit_config/launch/move_group.launch.py 	modified:   src/armv7_moveit_config/launch/moveit_rviz.launch.py 	modified:   src/armv7_moveit_config/launch/rsp.launch.py 	modified:   src/armv7_moveit_config/launch/setup_assistant.launch.py 	modified:   src/armv7_moveit_config/launch/spawn_controllers.launch.py 	modified:   src/armv7_moveit_config/launch/static_virtual_joint_tfs.launch.py 	modified:   src/armv7_moveit_config/launch/warehouse_db.launch.py 	new file:   src/armv7_moveit_config/package.xml

File: src/armv7_bringup/urdf/armv7_ethercat.ros2_control.xacro (robot description, xacro)
@@ -21,5 +21,5 @@
                   <param name="position">0</param>
                   <param name="mode_of_operation">8</param>
-                  <param name="slave_config">$(find armv7_moveit)/config/EUPH17_config.yaml</param>
+                  <param name="slave_config">$(find armv7_bringup)/config/EUPH17_config.yaml</param>
                 </ec_module>
             </joint>
@@ -36,5 +36,5 @@
                   <param name="position">1</param>
                   <param name="mode_of_operation">8</param>
-                  <param name="slave_config">$(find armv7_moveit)/config/EUPH17_config.yaml</param>
+                  <param name="slave_config">$(find armv7_bringup)/config/EUPH17_config.yaml</param>
                 </ec_module>
             </joint>
@@ -51,5 +51,5 @@
                   <param name="position">2</param>
                   <param name="mode_of_operation">8</param>
-                  <param name="slave_config">$(find armv7_moveit)/config/EUPH14_config.yaml</param>
+                  <param name="slave_config">$(find armv7_bringup)/config/EUPH14_config.yaml</param>
                 </ec_module>
             </joint>
@@ -66,5 +66,5 @@
                   <param name="position">3</param>
                   <param name="mode_of_operation">8</param>
-                  <param name="slave_config">$(find armv7_moveit)/config/EUPH14_config.yaml</param>
+                  <param name="slave_config">$(find armv7_bringup)/config/EUPH14_config.yaml</param>
                 </ec_module>
             </joint>
@@ -81,5 +81,5 @@
                   <param name="position">4</param>
                   <param name="mode_of_operation">8</param>
-                  <param name="slave_config">$(find armv7_moveit)/config/EUPH11_config.yaml</param>
+                  <param name="slave_config">$(find armv7_bringup)/config/EUPH11_config.yaml</param>
                 </ec_module>
             </joint>
@@ -96,5 +96,5 @@
                   <param name="position">5</param>
                   <param name="mode_of_operation">8</param>
-                  <param name="slave_config">$(find armv7_moveit)/config/EUPH11_config.yaml</param>
+                  <param name="slave_config">$(find armv7_bringup)/config/EUPH11_config.yaml</param>
                 </ec_module>
             </joint>
@@ -111,5 +111,5 @@
                   <param name="position">6</param>
                   <param name="mode_of_operation">8</param>
-                  <param name="slave_config">$(find armv7_moveit)/config/EUPH11_config.yaml</param>
+                  <param name="slave_config">$(find armv7_bringup)/config/EUPH11_config.yaml</param>
                 </ec_module>
             </joint>

File: src/armv7_description/urdf/armv7.urdf (robot description, URDF)
Before this commit: robot armv7, 8 links, 7 joints
Links:
- link base_link: geometry collision mesh filename=package://armv7_description/meshes/base_link.STL; visual mesh filename=package://armv7_description/meshes/base_link.STL
- link link1: geometry collision mesh filename=package://armv7_description/meshes/link1.STL; visual mesh filename=package://armv7_description/meshes/link1.STL
- link link2: geometry collision mesh filename=package://armv7_description/meshes/link2.STL; visual mesh filename=package://armv7_description/meshes/link2.STL
- link link3: geometry collision mesh filename=package://armv7_description/meshes/link3.STL; visual mesh filename=package://armv7_description/meshes/link3.STL
- link link4: geometry collision mesh filename=package://armv7_description/meshes/link4.STL; visual mesh filename=package://armv7_description/meshes/link4.STL
- link link5: geometry collision mesh filename=package://armv7_description/meshes/link5.STL; visual mesh filename=package://armv7_description/meshes/link5.STL
- link link6: geometry collision mesh filename=package://armv7_description/meshes/link6.STL; visual mesh filename=package://armv7_description/meshes/link6.STL
- link link7: geometry collision mesh filename=package://armv7_description/meshes/link7.STL; visual mesh filename=package://armv7_description/meshes/link7.STL
